Commit message: gripper tcp

File: ur_description/urdf/inc/ee_grain.xacro (robot description, xacro)
@@ -36,5 +36,5 @@
     <link name="${prefix}camera_tcp"/>
     <joint name="${prefix}gripper_joint" type="fixed">
-      <origin xyz="0.035955506 0 0.128865346" rpy="0 0 0"/>
+      <origin xyz="0.035955506 0 0.128865346" rpy="0 0 ${pi}"/>
       <parent link="${prefix}end_effector"/>
       <child link="${prefix}gripper_tcp"/>
@@ -42,5 +42,5 @@
     <link name="${prefix}gripper_tcp"/>
     <joint name="${prefix}gripper_s_joint" type="fixed">
-      <origin xyz="0 0 0.128865346" rpy="0 0 0"/>
+      <origin xyz="0 0 0.128865346" rpy="0 0 ${pi}"/>
       <parent link="${prefix}end_effector"/>
       <child link="${prefix}gripper_s_tcp"/>

Commit message: adjust tcp frames

File: ur_description/urdf/inc/ee_grain.xacro (robot description, xacro)
@@ -30,5 +30,5 @@
     <!-- TCP frames -->
     <joint name="${prefix}camera_joint" type="fixed">
-      <origin xyz="0.05715972 -0.105019695 0.049498274" rpy="${pi/2} 0 ${pi/2}"/>
+      <origin xyz="0.05715972 -0.105019695 0.049498274" rpy="0 ${-pi/2} ${pi}"/>
       <parent link="${prefix}end_effector"/>
       <child link="${prefix}camera_tcp"/>

Commit message: update tcp

File: ur_description/urdf/inc/ee_grain.xacro (robot description, xacro)
@@ -36,5 +36,5 @@
     <link name="${prefix}camera_tcp"/>
     <joint name="${prefix}gripper_joint" type="fixed">
-      <origin xyz="0.035955506 0 0.128865346" rpy="0 0 ${pi}"/>
+      <origin xyz="0.0 0.0 0.17644" rpy="0 0 ${pi}"/>
       <parent link="${prefix}end_effector"/>
       <child link="${prefix}gripper_tcp"/>

Commit message: moveit config

File: ur_description/urdf/inc/ee_grain.xacro (robot description, xacro)
@@ -41,10 +41,4 @@
     </joint>
     <link name="${prefix}gripper_tcp"/>
-    <joint name="${prefix}gripper_s_joint" type="fixed">
-      <origin xyz="0 0 0.128865346" rpy="0 0 ${pi}"/>
-      <parent link="${prefix}end_effector"/>
-      <child link="${prefix}gripper_s_tcp"/>
-    </joint>
-    <link name="${prefix}gripper_s_tcp"/>
   </xacro:macro>
 </robot>
