Commit message: zivid

File: ur10e_zivid_moveit_config/zivid_description/urdf/ur10e_zivid_macro.xacro (robot description, xacro)
@@ -40,5 +40,5 @@
       safety_k_position="${safety_k_position}"
     />
-    <xacro:include filename="$(find ur10e_zivid_moveit_config)/zivid_description/urdf/zivid.xacro"/>
+    <xacro:include filename="$(find ur10e_zivid_moveit_config)/zivid_description/urdf/zivid_macro.xacro"/>
     <xacro:end_effector prefix="" connected_to="flange"/>
   </xacro:macro>

File: ur10e_zivid_moveit_config/zivid_description/urdf/zivid_macro.xacro (robot description, xacro)
@@ -9,5 +9,5 @@
             <child link="${prefix}end_effector" />
             <!-- The tool is directly attached to the flange. -->
-            <origin rpy="0 0 ${-pi/2}" xyz="0 0 0" />
+            <origin rpy="${pi} ${-pi/2} 0" xyz="0 0 0" />
         </joint>
         <link name="${prefix}end_effector">
@@ -16,8 +16,8 @@
                     <!-- The path to the visual meshes in the package. -->
                     <mesh
-                        filename="$(find ur10e_zivid_moveit_config)/zivid_description/meshes/grain_ee_co.stl" />
+                        filename="package://ur10e_zivid_moveit_config/zivid_description/meshes/zivid_ee_v.stl" />
                 </geometry>
                 <material name="black">
-                    <color rgba="${0/255} ${0/255} ${0/255} 1.0" />
+                    <color rgba="${20/255} ${20/255} ${20/255} 1.0" />
                 </material>
             </visual>
@@ -26,5 +26,5 @@
                     <!-- The path to the collision meshes in the package. -->
                     <mesh
-                        filename="$(find ur10e_zivid_moveit_config)/zivid_description/meshes/zivid_ee_c.stl" />
+                        filename="package://ur10e_zivid_moveit_config/zivid_description/meshes/zivid_ee_c.stl" />
                 </geometry>
             </collision>
@@ -32,5 +32,5 @@
         <!-- TCP frames -->
         <joint name="${prefix}camera_joint" type="fixed">
-            <origin xyz="0.05715972 -0.105019695 0.049498274" rpy="0 ${-pi/2} ${pi}" />
+            <origin xyz="-0.057209 -0.043066 0.0545" rpy="${pi/2} 0 ${-pi/2}" />
             <parent link="${prefix}end_effector" />
             <child link="${prefix}camera_tcp" />
