Commit message: zivid urdf

File: ur10e_zivid_moveit_config/zivid_description/urdf/zivid_macro.xacro (robot description, xacro)
@@ -9,5 +9,5 @@
             <child link="${prefix}end_effector" />
             <!-- The tool is directly attached to the flange. -->
-            <origin rpy="${pi} ${-pi/2} 0" xyz="0 0 0" />
+            <origin rpy="-1.5705926535266412 -0.7853983060537703 -1.5710843642474572" xyz="0 0 0" />
         </joint>
         <link name="${prefix}end_effector">
@@ -19,5 +19,5 @@
                 </geometry>
                 <material name="black">
-                    <color rgba="${20/255} ${20/255} ${20/255} 1.0" />
+                    <color rgba="${50/255} ${50/255} ${50/255} 1.0" />
                 </material>
             </visual>
@@ -32,5 +32,5 @@
         <!-- TCP frames -->
         <joint name="${prefix}camera_joint" type="fixed">
-            <origin xyz="-0.057209 -0.043066 0.0545" rpy="${pi/2} 0 ${-pi/2}" />
+            <origin xyz="0.057209 0.043066 0.0795" rpy="${pi/2} 0 ${pi/2}" />
             <parent link="${prefix}end_effector" />
             <child link="${prefix}camera_tcp" />
