Commit message: ur10e_ka

File: ur10e_ka_moveit_config/ka_description/urdf/ka_macro.xacro (robot description, xacro)
@@ -9,5 +9,5 @@
             <child link="${prefix}end_effector" />
             <!-- The tool is directly attached to the flange. -->
-            <origin rpy="0 ${pi/2} 0" xyz="0 0 0" />
+            <origin rpy="0 ${-pi/2} ${pi}" xyz="0 0 0" />
         </joint>
         <link name="${prefix}end_effector">

Commit message: ur10e_ka

File: ur10e_ka_moveit_config/ka_description/urdf/ka_macro.xacro (robot description, xacro)
@@ -31,10 +31,16 @@
         </link>
         <!-- TCP frames -->
-        <joint name="${prefix}camera_joint" type="fixed">
-            <origin xyz="0.057209 0.043066 0.0795" rpy="${pi/2} 0 ${pi/2}" />
+        <joint name="${prefix}depth_camera_joint" type="fixed">
+            <origin xyz="0.111986021427 6.69550452272e-8 2.22519248532e-02" rpy="-1.675516081915675 1.6790457912918555e-12 -1.570796326781967" />
             <parent link="${prefix}end_effector" />
-            <child link="${prefix}camera_tcp" />
+            <child link="${prefix}depth_camera_tcp" />
         </joint>
-        <link name="${prefix}camera_tcp" />
+        <link name="${prefix}depth_camera_tcp" />
+        <joint name="${prefix}rgb_camera_joint" type="fixed">
+            <origin xyz="0.10554133441 -3.19999999972e-02 1.94659300526e-02" rpy="-1.5707963267928968 0.0 -1.5707963267808966" />
+            <parent link="${prefix}end_effector" />
+            <child link="${prefix}rgb_camera_tcp" />
+        </joint>
+        <link name="${prefix}rgb_camera_tcp" />
     </xacro:macro>
 </robot>
